File: kicad/rtlm/rtlm.kicad_sch (KiCad schematic)
At the start: 37 parts, among them IC1 ESP32-S3FN8, IC2 TPS25940ARVCR, J1 USB_C_Receptacle_USB2.0_16P, J2 Conn_01x02, Q1 DMP2035U-7, U1 TPS62130A, U2 TPS2116DRL

Commit message: feat: start LoRa, finish basic ESP32 schematic
Parts:
- added C14, C15: 100nf, symbol Device:C
- added C16: 10µf, symbol Device:C
- added C17, C18: 1µf, symbol Device:C
- added C19, C20: 16pf, symbol Device:C
- added C21, C23: 100nf, Package_DFN_QFN:QFN-24-1EP_4x4mm_P0.5mm_EP2.6x2.6mm, symbol Device:C
- added C22: 470nf, Package_DFN_QFN:QFN-24-1EP_4x4mm_P0.5mm_EP2.6x2.6mm, symbol Device:C
- added C24: 10pf, Package_DFN_QFN:QFN-24-1EP_4x4mm_P0.5mm_EP2.6x2.6mm, symbol Device:C
- added IC3: PE4259, SOT65P210X110-6N, symbol SamacSys_Parts:PE4259
- added J3: UART_DEBUG_3V3, Package_TO_SOT_SMD:Texas_DRT-3, symbol Connector_Generic:Conn_01x03
- added L2: 2nH, symbol Device:L
- added L3: 24nh, symbol Device:L
- added L4: 15µh, symbol Device:L
- added R16, R17, R18, R19, R21: 10k, symbol Device:R
- added R20: 499, symbol Device:R
- added R22: 220, symbol Device:R
- added SW1, SW2: SW_Push, Package_SON:WSON-8-1EP_6x5mm_P1.27mm_EP3.4x4mm, symbol Switch:SW_Push
- added U3: TPD2EUSB30, Package_TO_SOT_SMD:Texas_DRT-3, symbol Power_Protection:TPD2EUSB30
- added U4: SX1262IMLTRT, Package_DFN_QFN:QFN-24-1EP_4x4mm_P0.5mm_EP2.6x2.6mm, symbol RF:SX1262IMLTRT
- added Y1: 40MHz, Crystal:Crystal_SMD_SeikoEpson_FA128-4Pin_2.0x1.6mm, symbol Device:Crystal_GND24
- added Y2: TG2520SMN 32.0000M-MCGNNM3, Oscillator:Oscillator_SMD_SeikoEpson_TG2520SMN-xxx-xxxxxx-4Pin_2.5x2.0mm, symbol Oscillator:TG2520SMN-xx.xxxxxxMhz-xxxxNM
Connections:
- net +3.3V: now also IC1.55 (VDDA_1), IC1.56 (VDDA_2), C14.2, C15.2, C16.1, C21.1, L2.1, R16.2, R17.2, R21.2, U4.1 (VDD_IN), U4.10 (VBAT), U4.11 (VBAT_IO)
- net GND: now also C14.1, C15.1, C16.2, C17.1, C18.1, C19.1, C20.1, C21.2, C22.1, C23.1, J3.1 (Pin_1), R18.1, R19.1, SW1.2, SW2.2, U3.3 (GND), U4.2 (GND), U4.20 (GND), U4.25 (GND), U4.5 (GND), U4.8 (GND), Y1.2 (G), Y1.4 (G), Y2.2 (GND)
- net USB_DM: now also U3.2 (D-)
- net USB_DP: now also U3.1 (D+)
- net LORA_BUSY: now reaches IC1.10 (GPIO5)
- net LORA_BUSY: now also U4.14 (BUSY)
- net LORA_IRQ: now reaches IC1.11 (GPIO6)
- net LORA_IRQ: now also U4.13 (DIO1)
- net LORA_CS: now reaches IC1.15 (GPIO10)
- net LORA_CS: now also R21.1, U4.19 (NSS)
- net LORA_MOSI: now reaches IC1.16 (GPIO11)
- net LORA_MOSI: now also U4.17 (MOSI)
- net LORA_SCK: now reaches IC1.17 (GPIO12)
- net LORA_SCK: now also U4.18 (SCK)
- net LORA_MISO: now reaches IC1.18 (GPIO13)
- net LORA_MISO: now also U4.16 (MISO)
- net at IC1.2 (VDD3P3_1): now also IC1.3 (VDD3P3_2), C17.2, L2.2
- net at IC1.4 (CHIP_PU): now also C18.2, R16.1, SW1.1
- net ESP_U0TXD: now reaches IC1.49 (U0TXD)
- net ESP_U0TXD: now also R20.2
- net at IC1.5 (GPIO0): now also R17.1, SW2.1
- net ESP_U0RXD: now reaches IC1.50 (U0RXD)
- net ESP_U0RXD: now also J3.3 (Pin_3)
- net at IC1.51 (GPIO45): now also R19.2
- net at IC1.52 (GPIO46): now also R18.2
- net ESP_XTAL_P: now reaches IC1.53 (XTAL_N)
- net ESP_XTAL_P: now also IC1.54 (XTAL_P), L3.1
- net LORA_RESET: now reaches IC1.9 (GPIO4)
- net LORA_RESET: now also U4.15 (~{RESET})
- new net: C20.2, L3.2, Y1.1
- new net: C22.2, L4.1, U4.7 (VREG)
- new net: R22.1, Y2.3 (OUT)
- new net: C24.1, R22.2
- new net: J3.2 (Pin_2), R20.1
- new net: L4.2, U4.9 (DCC_SW)
- new net: C23.2, U4.6 (DIO3), Y2.4 (Vcc)
- new net ESP_XTAL_N: C19.2, Y1.3
- new net LORA_XTA: C24.2, U4.3 (XTA)
- no-connect marks 6 -> 8
Other:
- note added: "BOOT"
- note added: "RESET"
- moved on the sheet: C1, C10, C11, C12, C13, C2, C3, C4, C5, C6, IC1, J1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

Commit message: feat: basic LoRa module complete
Parts:
- added C25: 1nf, symbol Device:C
- added C26: 100nf, symbol Device:C
- added C27, C32: 39pf, symbol Device:C
- added C28: 2.4pf, symbol Device:C
- added C29, C37: 1.8pf, symbol Device:C
- added C30, C31: 3.3pf, symbol Device:C
- added C33: 47nf, symbol Device:C
- added C34: 47pf, symbol Device:C
- added C35: 3pf, symbol Device:C
- added C36: 5.6pf, symbol Device:C
- added C38: 1µf, symbol Device:C
- added J4: LORA_ANT, Connector_Coaxial:U.FL_Hirose_U.FL-R-SMT-1_Vertical, symbol Connector:Conn_Coaxial
- added L5: 15nH, symbol Device:L
- added L6: 9.1nh, symbol Device:L
- added L7: 2.5nh, symbol Device:L
- added L8: 4.7nh, symbol Device:L
- added L9: 47nh, symbol Device:L
- added R23: 220, symbol Device:R
- added R24: 2.2k, symbol Device:R
- added R25: 0, symbol Device:R
Connections:
- net +3.3V: now also C38.1
- net GND: now also IC3.2 (GND), C25.1, C26.1, C29.1, C30.2, C31.2, C33.2, C34.2, C36.2, C37.2, C38.2, J4.2 (Ext), R24.1
- net at U4.12 (DIO2): now also R23.2
- net at U4.21 (RFI_P): now also C29.2, L5.2
- net LORA_RFI_N: now reaches U4.22 (RFI_N)
- net LORA_RFI_N: now also C28.2, L5.1
- net LORA_RFO: now reaches U4.23 (RFO)
- net LORA_RFO: now also R25.1
- net LORA_VR_PA: now reaches U4.24 (VR_PA)
- net LORA_VR_PA: now also C33.1, C34.1, L9.2
- net LORA_3V0: now reaches C23.2, U4.6 (DIO3), Y2.4 (Vcc)
- net LORA_3V0: now also IC3.6 (~{CTRL_OR_VDD}), C26.2
- net at IC3.1 (RF1): now also C37.1, L8.2
- net at IC3.3 (RF2): now also C28.1
- net at IC3.4 (CTRL): now also C25.2, R23.1, R24.2
- net at IC3.5 (RFC): now also C27.2
- new net: C27.1, C31.1, L6.2
- new net: C32.2, L8.1
- new net: C35.1, L7.1, L9.1, R25.2
- new net: C30.1, J4.1 (In), L6.1
- new net: C32.1, C35.2, C36.1, L7.2
Other:
- moved on the sheet: C23, C24, IC3, R22, Y2

Commit message: feat: basic sensor support
Parts:
- added C39, C46: 100nf, symbol Device:C
- added C40, C41, C43, C45: 1nf, symbol Device:C
- added C42: 1µf, SOT95P280X145-6N, symbol Device:C
- added C44: 10µf, symbol Device:C
- added C47: 470nf, Package_TO_SOT_SMD:SOT-23, symbol Device:C
- added C48: 1µf, symbol Device:C
- added D2, D4, D6, D8: PESD5V0S1UL, Diode_SMD:D_SOD-882, symbol Diode:PESD5V0S1UL
- added D3, D5, D7, D9: BAT54S, Package_TO_SOT_SMD:SOT-23, symbol Diode:BAT54S
- added IC4: TPS2553DBVR, SOT95P280X145-6N, symbol SamacSys_Parts:TPS2553DBVR
- added J5: PULSE_1, symbol Connector_Generic:Conn_01x04
- added J6: PULSE_2, symbol Connector_Generic:Conn_01x04
- added J7: PULSE_3, symbol Connector_Generic:Conn_01x04
- added J8: PULSE_4, symbol Connector_Generic:Conn_01x04
- added R26, R29, R31, R33: 1k, symbol Device:R
- added R27, R28, R30, R32: 4.7k, symbol Device:R
- added R34: 133k, Package_LCC:PLCC-84_29.3x29.3mm_P1.27mm, symbol Device:R
- added R35: 100k, symbol Device:R
- added R36: 10k, symbol Device:R
- added U5: SN74LVC14ADR, Package_SO:SOIC-14_3.9x8.7mm_P1.27mm, symbol 74xx:74HC14
- added U6: MCP3208, Package_DFN_QFN:QFN-20-1EP_5x5mm_P0.65mm_EP3.35x3.35mm, symbol Analog_ADC:MCP3208
- added U7: REF3025, Package_TO_SOT_SMD:SOT-23, symbol Reference_Voltage:REF3025
Connections:
- net +3.3V: now also C39.1, C46.1, C47.1, D3.2 (K), D5.2 (K), D7.2 (K), D9.2 (K), R27.2, R28.2, R30.2, R32.2, R36.2, U5.14 (VCC), U6.16 (Vdd), U7.1 (IN)
- net 5V_SYS: now also C42.2, IC4.1 (IN)
- net GND: now also C39.2, C40.2, C41.2, C42.1, C43.2, C44.1, C45.2, C46.2, C47.2, C48.2, D2.2 (A), D3.1 (A), D4.2 (A), D5.1 (A), D6.2 (A), D7.1 (A), D8.2 (A), D9.1 (A), IC4.2 (GND), J5.1 (Pin_1), J6.1 (Pin_1), J7.1 (Pin_1), J8.1 (Pin_1), R34.2, R35.2, U5.11, U5.13, U5.7 (GND), U6.14 (AGND), U6.9 (DGND), U7.3 (GND)
- net LORA_MISO: now also U6.12 (Dout)
- net LORA_MOSI: now also U6.11 (Din)
- net ESP_RESET: now reaches C18.2, IC1.4 (CHIP_PU), R16.1, SW1.1
- net ESP_BOOT: now reaches IC1.5 (GPIO0), R17.1, SW2.1
- net PULSE_1: now reaches IC1.12 (GPIO7)
- net PULSE_1: now also U5.2
- net PULSE_2: now reaches IC1.13 (GPIO8)
- net PULSE_2: now also U5.4
- net PULSE_3: now reaches IC1.14 (GPIO9)
- net PULSE_3: now also U5.6
- net PULSE_4: now reaches IC1.19 (GPIO14)
- net PULSE_4: now also U5.8
- net ADC_CS: now reaches IC1.23 (GPIO17)
- net ADC_CS: now also U6.10 (~{CS}/SHDN)
- net PULSE_PWR_EN: now reaches IC1.6 (GPIO1)
- net PULSE_PWR_EN: now also IC4.3 (EN), R35.1
- net PULSE_PWR_FAULT: now reaches IC1.7 (GPIO2)
- net PULSE_PWR_FAULT: now also IC4.4 (~{FAULT}), R36.1
- new net: C43.1, D7.3 (COM), R31.2, U5.5
- new net: C40.1, D3.3 (COM), R26.2, U5.1
- new net: IC4.5 (ILIM), R34.1
- new net: C45.1, D9.3 (COM), R33.2, U5.9
- new net: C41.1, D5.3 (COM), R29.2, U5.3
- new net 5V_PULSE: C44.2, IC4.6 (OUT), J5.2 (Pin_2), J6.2 (Pin_2), J7.2 (Pin_2), J8.2 (Pin_2)
- new net ADC_VREF_2V5: C48.1, U6.15 (Vref), U7.2 (OUT)
- new net PULSE1_RAW: D2.1 (K), J5.3 (Pin_3), R26.1, R27.1
- new net PULSE2_RAW: D4.1 (K), J6.3 (Pin_3), R28.1, R29.1
- new net PULSE3_RAW: D6.1 (K), J7.3 (Pin_3), R30.1, R31.1
- new net PULSE4_RAW: D8.1 (K), J8.3 (Pin_3), R32.1, R33.1
- no-connect marks 8 -> 14
Other:
- moved on the sheet: C10, C18, R16, R17, SW1, SW2

Commit message: feat: status LEDs, more sensor ports, start CAN, SD card
Parts:
- added C49, C51, C52, C53: 100nf, symbol Device:C
- added C50, C58, C59, C61: 100nf, SOIC127P600X175-14N, symbol Device:C
- added C54, C55, C56, C57: 10nf, SOIC127P600X175-14N, symbol Device:C
- added C60: 10µf, SOIC127P600X175-14N, symbol Device:C
- added C62, C63: 100nf, SOIC127P600X175-8N, symbol Device:C
- added C65: 10µf, symbol Device:C
- added C66: 1µf, SOT95P280X145-6N, symbol Device:C
- added D10, D11, D12, D13, D14, D15, D16, D17: PESD5V0L1UA, Diode_SMD:D_SOD-323, symbol SamacSys_Parts:PESD5V0L1UA
- added D18, D22, D23, D24: LED, LED_SMD:LED_0603_1608Metric, symbol Device:LED
- added D19: PESD2CAN, Package_TO_SOT_SMD:SOT-23, symbol SamacSys_Parts:PESD2CAN
- added IC5, IC6: TLV9004IDR, SOIC127P600X175-14N, symbol SamacSys_Parts:TLV9004IDR
- added IC7: TCAN1042HGVDR, Package_SO:SOIC-8_3.9x4.9mm_P1.27mm, symbol SamacSys_Parts:TCAN1042HGVDR
- added IC8: TPS2553DBVR, SOT95P280X145-6N, symbol SamacSys_Parts:TPS2553DBVR
- added J10: TEMP_2, symbol Connector_Generic:Conn_01x04
- added J11: TEMP_3, symbol Connector_Generic:Conn_01x04
- added J12: TEMP_4, symbol Connector_Generic:Conn_01x04
- added J13: ANALOG_1, symbol Connector_Generic:Conn_01x04
- added J14: ANALOG_2, symbol Connector_Generic:Conn_01x04
- added J15: ANALOG_3, symbol Connector_Generic:Conn_01x04
- added J16: ANALOG_4, symbol Connector_Generic:Conn_01x04
- added J17: DM3AT-SF-PEJM5, Connector_Card:microSD_HC_Hirose_DM3AT-SF-PEJM5, symbol Connector:Micro_SD_Card_Det_Hirose_DM3AT
- added J18: CAN_EXPANSION, RF_Module:nRF24L01_Breakout, symbol Connector:Conn_01x06_Pin
- added J9: TEMP_1, symbol Connector_Generic:Conn_01x04
- added JP1: CAN_TERM, PESD2CAN, symbol Jumper:Jumper_2_Open
- added R37, R38, R41, R43, R45, R52, R54, R57, R60, R74, R79: 10k, symbol Device:R
- added R39, R42, R44, R46, R51, R55, R58, R61: 4.7k, symbol Device:R
- added R40, R47, R48, R49, R62, R63, R64, R65: 47, symbol Device:R
- added R50, R53, R56, R59: 12k, symbol Device:R
- added R66: 20k, SOD2512X110N, symbol Device:R
- added R67, R68, R69, R70, R71, R72: 10k, SOD2512X110N, symbol Device:R
- added R73: 33, symbol Device:R
- added R75, R76, R77, R78: 1k, symbol Device:R
- added R80: 120, symbol Device:R
- added R81: 133k, symbol Device:R
- added R85: 2.2k, symbol Device:R
- U7: value REF3025 -> REF3025AIDBZR
Connections:
- net +3.3V: now also C50.1, C58.1, C60.1, C61.1, C63.1, IC5.4 (V+), IC6.4 (V+), IC7.5 (VIO), J17.4 (VDD), R37.1, R68.2, R69.2, R70.2, R71.2, R72.2, R74.2, R75.1, R79.2
- net 5V_PULSE: now also J13.2 (Pin_2), J14.2 (Pin_2), J15.2 (Pin_2), J16.2 (Pin_2), R66.1
- net 5V_SYS: now also C62.1, C66.2, IC7.3 (VCC), IC8.1 (IN)
- net ADC_CS: now also R37.2
- net ADC_VREF_2V5: now also R38.1, R41.1, R43.1, R45.1
- net GND: now also C49.2, C50.2, C51.2, C52.2, C53.2, C54.2, C55.2, C56.2, C57.2, C58.2, C59.2, C60.2, C61.2, C62.2, C63.2, C65.1, C66.1, D10.2 (A), D11.2 (A), D12.2 (A), D13.2 (A), D14.2 (A), D15.2 (A), D16.2 (A), D17.2 (A), D18.1 (K), D19.3 (I/O_3), D22.1 (K), D23.1 (K), D24.1 (K), IC5.11 (V-), IC6.11 (V-), IC7.2 (GND), IC8.2 (GND), J10.1 (Pin_1), J11.1 (Pin_1), J12.1 (Pin_1), J13.1 (Pin_1), J14.1 (Pin_1), J15.1 (Pin_1), J16.1 (Pin_1), J17.10 (DET_A), J17.6 (VSS), J17.SH (SHIELD), J18.1 (Pin_1), J9.1 (Pin_1), R52.2, R54.2, R57.2, R60.2, R67.1, R81.2, R85.2
- net LORA_SCK: now also U6.13 (CLK)
- net TEMP1_ADC: now reaches U6.1 (CH0)
- net TEMP1_ADC: now also R40.1
- net TEMP2_ADC: now reaches U6.2 (CH1)
- net TEMP2_ADC: now also R47.1
- net TEMP3_ADC: now reaches U6.3 (CH2)
- net TEMP3_ADC: now also R48.1
- net TEMP4_ADC: now reaches U6.4 (CH3)
- net TEMP4_ADC: now also R49.1
- net ANALOG1_ADC: now reaches U6.5 (CH4)
- net ANALOG1_ADC: now also R62.1
- net ANALOG2_ADC: now reaches U6.6 (CH5)
- net ANALOG2_ADC: now also R63.1
- net ANALOG3_ADC: now reaches U6.7 (CH6)
- net ANALOG3_ADC: now also R65.1
- net ANALOG4_ADC: now reaches U6.8 (CH7)
- net ANALOG4_ADC: now also R64.1
- net LED_LOG: now reaches IC1.21 (XTAL_32K_P)
- net LED_LOG: now also R78.1
- net LED_RADIO: now reaches IC1.22 (XTAL_32K_N)
- net LED_RADIO: now also R77.1
- net SENSOR_5V_MON: now reaches IC1.24 (GPIO18)
- net SENSOR_5V_MON: now also C59.1, R66.2, R67.2
- net SD_DETECT: now reaches IC1.27 (GPIO21)
- net SD_DETECT: now also J17.9 (DET_B), R74.1
- net CAN_PWR_EN: now reaches IC1.28 (SPICS1)
- net CAN_PWR_EN: now also IC8.3 (EN), R85.1
- net LED_FAULT: now reaches IC1.38 (GPIO33)
- net LED_FAULT: now also R76.1
- net CAN_TX: now reaches IC1.39 (GPIO34)
- net CAN_TX: now also IC7.1 (TXD)
- net CAN_RX: now reaches IC1.40 (GPIO35)
- net CAN_RX: now also IC7.4 (RXD)
- net CAN_STB: now reaches IC1.41 (GPIO36)
- net CAN_STB: now also IC7.8 (STB), R79.1
- net SD_D3: now reaches IC1.42 (GPIO37)
- net SD_D3: now also J17.2 (DAT3/CD), R69.1
- net at IC1.43 (GPIO38): now also R73.1
- net SD_CMD: now reaches IC1.44 (MTCK)
- net SD_CMD: now also J17.3 (CMD), R70.1
- net SD_D0: now reaches IC1.45 (MTDO)
- net SD_D0: now also J17.7 (DAT0), R71.1
- net SD_D1: now reaches IC1.47 (MTDI)
- net SD_D1: now also J17.8 (DAT1), R72.1
- net SD_D2: now reaches IC1.48 (MTMS)
- net SD_D2: now also J17.1 (DAT2), R68.1
- net PULSE_PWR_FAULT renamed SENSOR_PWR_FAULT
- net SENSOR_PWR_FAULT: now also IC8.4 (~{FAULT})
- new net: IC5.1 (OUT1), IC5.2 (IN1-), R40.2
- new net: IC6.13 (IN4-), IC6.14 (OUT4), R64.2
- new net: R50.2, R51.1, R52.1
- new net: D24.2 (A), R78.2
- new net: JP1.2 (B), R80.2
- new net: R59.2, R60.1, R61.1
- new net: IC6.1 (OUT1), IC6.2 (IN1-), R62.2
- new net: IC6.6 (IN2-), IC6.7 (OUT2), R63.2
- new net: IC6.8 (OUT3), IC6.9 (IN3-), R65.2
- new net: IC5.6 (IN2-), IC5.7 (OUT2), R47.2
- new net: R53.2, R54.1, R55.1
- new net: D23.2 (A), R77.2
- new net: IC5.8 (OUT3), IC5.9 (IN3-), R48.2
- new net: IC8.5 (ILIM), R81.1
- new net: R56.2, R57.1, R58.1
- new net: D22.2 (A), R76.2
- new net: D18.2 (A), R75.2
- new net: IC5.13 (IN4-), IC5.14 (OUT4), R49.2
- new net 5V_CAN: C65.2, IC8.6 (OUT), J18.2 (Pin_2)
- new net ANALOG1_FILTERED: C54.1, IC6.3 (IN1+), R51.2
- new net ANALOG1_RAW: D14.1 (K), J13.3 (Pin_3), R50.1
- new net ANALOG2_FILTERED: C55.1, IC6.5 (IN2+), R55.2
- new net ANALOG2_RAW: D15.1 (K), J14.3 (Pin_3), R53.1
- new net ANALOG3_FILTERED: C56.1, IC6.10 (IN3+), R58.2
- new net ANALOG3_RAW: D16.1 (K), J15.3 (Pin_3), R56.1
- new net ANALOG4_FILTERED: C57.1, IC6.12 (IN4+), R61.2
- new net ANALOG4_RAW: D17.1 (K), J16.3 (Pin_3), R59.1
- new net CAN_H: D19.1 (I/O_1), IC7.7 (CANH), J18.3 (Pin_3), R80.1
- new net CAN_L: D19.2 (I/O_2), IC7.6 (CANL), J18.4 (Pin_4), JP1.1 (A)
- new net SD_CLK: J17.5 (CLK), R73.2
- new net TEMP1_FILTERED: C49.1, IC5.3 (IN1+), R39.2
- new net TEMP1_RAW: D10.1 (K), J9.3 (Pin_3), R38.2, R39.1
- new net TEMP2_FILTERED: C51.1, IC5.5 (IN2+), R42.2
- new net TEMP2_RAW: D11.1 (K), J10.3 (Pin_3), R41.2, R42.1
- new net TEMP3_FILTERED: C52.1, IC5.10 (IN3+), R44.2
- new net TEMP3_RAW: D12.1 (K), J11.3 (Pin_3), R43.2, R44.1
- new net TEMP4_FILTERED: C53.1, IC5.12 (IN4+), R46.2
- new net TEMP4_RAW: D13.1 (K), J12.3 (Pin_3), R45.2, R46.1
- no-connect marks 14 -> 28
Other:
- note added: "FAULT"
- note added: "LOG"
- note added: "POWER"
- note added: "RADIO"
- moved on the sheet: C11, U3

Commit message: feat: battery voltage sensing, sensor LEDs, start fixing footprint issues
Parts:
- added C64, C69: 1µf, Package_SO:SOIC-16W_7.5x10.3mm_P1.27mm, symbol Device:C
- added C67, C70, C72: 1nf, Package_SO:SOIC-16W_7.5x10.3mm_P1.27mm, symbol Device:C
- added C68, C71, C73: 100nf, Package_SO:SOIC-16W_7.5x10.3mm_P1.27mm, symbol Device:C
- added C74, C75: 10nf, Package_SO:SOIC-16W_7.5x10.3mm_P1.27mm, symbol Device:C
- added C76: 100nf, symbol Device:C
- added C77: 1µf, symbol Device:C
- added D20, D21, D25, D26, D27, D28, D29, D30, D31, D32, D33, D34: LED, symbol Device:LED
- added IC9: TLC59116IPWR, SOP65P640X120-28N, symbol SamacSys_Parts:TLC59116IPWR
- added J19: BATTERY_IN, Connector_AMASS:AMASS_XT60PW-F_1x02_P7.20mm_Horizontal, symbol Connector_Generic:Conn_01x02
- added J20: BATTERY_OUT, Connector_AMASS:AMASS_XT60PW-M_1x02_P7.20mm_Horizontal, symbol Connector_Generic:Conn_01x02
- added R82, R83: 499k, symbol Device:R
- added R84: 8.2k, symbol Device:R
- added R86, R87: 470, symbol Device:R
- added R88, R89: 4.7k, Package_SO:TSSOP-10_3x3mm_P0.5mm, symbol Device:R
- added R90: 1k, symbol Device:R
- added R91: 10k, SOP65P640X120-28N, symbol Device:R
- added R92: 1.8k, SOP65P640X120-28N, symbol Device:R
- added U8: AMC3330, Package_SO:SOIC-16W_7.5x10.3mm_P1.27mm, symbol Isolator_Analog:AMC3330
- added U9: ADS1115IDGS, Package_SO:TSSOP-10_3x3mm_P0.5mm, symbol Analog_ADC:ADS1115IDGS
- C42, C66: footprint SOT95P280X145-6N -> Capacitor_SMD:C_0603_1608Metric
- C50, C54, C55, C56, C57, C58, C59, C60, C61: footprint SOIC127P600X175-14N -> Capacitor_SMD:C_0603_1608Metric
- C62, C63: footprint SOIC127P600X175-8N -> Capacitor_SMD:C_0603_1608Metric
Connections:
- net +3.3V: now also C64.2, C67.2, C73.2, C76.1, C77.1, D20.2 (A), D21.2 (A), D25.2 (A), D26.2 (A), D27.2 (A), D28.2 (A), D29.2 (A), D30.2 (A), D31.2 (A), D32.2 (A), D33.2 (A), D34.2 (A), IC9.28 (VCC), R88.2, R89.2, R91.2, U8.12 (VDD), U9.8 (VDD)
- net GND: now also C64.1, C67.1, C68.2, C73.1, C76.2, C77.2, IC9.10 (GND_1), IC9.19 (GND_2), IC9.2 (A0), IC9.24 (GND_3), IC9.3 (A1), IC9.4 (A2), IC9.5 (A3), R92.2, U8.15 (DCDC_GND), U8.9 (GND), U9.1 (ADDR), U9.3 (GND), U9.6 (AIN2), U9.7 (AIN3)
- net I2C_SCL: now reaches IC1.36 (SPICLK_N)
- net I2C_SCL: now also IC9.26 (SCL), R88.1, U9.10 (SCL)
- net I2C_SDA: now reaches IC1.37 (SPICLK_P)
- net I2C_SDA: now also IC9.27 (SDA), R89.1, U9.9 (SDA)
- new net: IC9.1 (REXT), R92.1
- new net: C74.1, R83.2, R84.2, R90.1
- new net: IC9.25 (~{RESET}), R91.1
- new net: R86.1, U8.11 (OUTP)
- new net: C75.1, R86.2, U9.4 (AIN0)
- new net: R87.1, U8.10 (OUTN)
- new net: C75.2, R87.2, U9.5 (AIN1)
- new net: R82.2, R83.1
- new net HLDO_OUT: C71.2, C72.2, U8.5 (HLDO_OUT)
- new net LED_OUT0: D20.1 (K), IC9.6 (~{OUT0})
- new net LED_OUT1: D21.1 (K), IC9.7 (~{OUT1})
- new net LED_OUT10: D33.1 (K), IC9.17 (~{OUT10})
- new net LED_OUT11: D34.1 (K), IC9.18 (~{OUT11})
- new net LED_OUT2: D25.1 (K), IC9.8 (~{OUT2})
- new net LED_OUT3: D26.1 (K), IC9.9 (~{OUT3})
- new net LED_OUT4: D27.1 (K), IC9.11 (~{OUT4})
- new net LED_OUT5: D28.1 (K), IC9.12 (~{OUT5})
- new net LED_OUT6: D29.1 (K), IC9.13 (~{OUT6})
- new net LED_OUT7: D30.1 (K), IC9.14 (~{OUT7})
- new net LED_OUT8: D31.1 (K), IC9.15 (~{OUT8})
- new net LED_OUT9: D32.1 (K), IC9.16 (~{OUT9})
- new net PACK_NEG: C69.1, C70.1, C71.1, C72.1, C74.2, J19.1 (Pin_1), J20.1 (Pin_1), R84.1, U8.2 (DCDC_HGND), U8.7 (INN), U8.8 (HGND)
- new net PACK_POS: J19.2 (Pin_2), J20.2 (Pin_2), R82.1
- new net PACK_V_SENSE: R90.2, U8.6 (INP)
- new net VMON_DCDC_IN: C68.1, U8.13 (LDO_OUT), U8.16 (DCDC_IN)
- new net VMON_ISO_SUPPLY: C69.2, C70.2, U8.1 (DCDC_OUT), U8.3 (HLDO_IN)
- no-connect marks 28 -> 41
Other:
- moved on the sheet: C39, C40, C41, C43, C45, C49, C50, C51, C52, C53, C54, C55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

Commit message: feat: RTC, cleanup footprints
Parts:
- added BT1: CR2032, Battery:BatteryHolder_Keystone_1060_1x2032, symbol Device:Battery_Cell
- added C78, C79: 100nf, symbol Device:C
- added R93: 10k, symbol Device:R
- added R94: 1k, symbol Device:R
- added U10: RV-3028-C7, Package_SON:MicroCrystal_C7_SON-8_1.5x3.2mm_P0.9mm, symbol Timer_RTC:RV-3028-C7
- R11, R12: footprint QFN50P300X400X80-21N -> (none)
- R66, R67, R68, R69, R70, R71, R72: footprint SOD2512X110N -> (none)
- R91, R92: footprint SOP65P640X120-28N -> (none)
Connections:
- net +3.3V: now also C78.2, U10.7 (VDD)
- net GND: now also BT1.2 (-), C78.1, C79.1, R93.1, U10.5 (VSS)
- net I2C_SCL: now also U10.3 (SCL)
- net I2C_SDA: now also U10.4 (SDA)
- new net: BT1.1 (+), R94.2
- new net: R93.2, U10.8 (EVI)
- new net RTC_BACKUP: C79.2, R94.1, U10.6 (VBACKUP)
- no-connect marks 41 -> 43

Commit message: feat: finish schematic, fix footprints and verify components
Parts:
- C1: footprint Package_DFN_QFN:VQFN-16-1EP_3x3mm_P0.5mm_EP1.68x1.68mm_ThermalVias -> Capacitor_SMD:C_0805_2012Metric
- C10, C11, C12, C13, C14, C15, C17, C18, C19, C20, C38, C39, C4, C40, C41, C43, C45, C46, C48, C49, C51, C52, C53, C6, C7, C76, C77, C78, C79, C8, C9: footprint (none) -> Capacitor_SMD:C_0603_1608Metric
- C16, C44, C65: footprint (none) -> Capacitor_SMD:C_0805_2012Metric
- C2: footprint Package_DFN_QFN:VQFN-16-1EP_3x3mm_P0.5mm_EP1.68x1.68mm_ThermalVias -> Capacitor_SMD:C_0603_1608Metric
- C21, C22, C23, C24: footprint Package_DFN_QFN:QFN-24-1EP_4x4mm_P0.5mm_EP2.6x2.6mm -> Capacitor_SMD:C_0402_1005Metric
- C25, C26, C27, C28, C29, C30, C31, C32, C33, C34, C35, C36, C37: footprint (none) -> Capacitor_SMD:C_0402_1005Metric
- C3: footprint Package_DFN_QFN:VQFN-16-1EP_3x3mm_P0.5mm_EP1.68x1.68mm_ThermalVias -> Capacitor_SMD:C_1206_3216Metric
- C47: footprint Package_TO_SOT_SMD:SOT-23 -> Capacitor_SMD:C_0603_1608Metric
- C5: footprint Package_TO_SOT_SMD:SOT-583-8 -> Capacitor_SMD:C_0603_1608Metric
- C60: footprint Capacitor_SMD:C_0603_1608Metric -> Capacitor_SMD:C_0805_2012Metric
- C64, C67, C71, C72: footprint Package_SO:SOIC-16W_7.5x10.3mm_P1.27mm -> Capacitor_SMD:C_1206_3216Metric
- C68, C69, C70, C73, C74, C75: footprint Package_SO:SOIC-16W_7.5x10.3mm_P1.27mm -> Capacitor_SMD:C_0603_1608Metric
- D1: value 5.6V -> BZT52C5V6; footprint (none) -> Diode_SMD:D_SOD-123
- D20, D21, D25, D26, D27, D28, D29, D30, D31, D32, D33, D34: footprint (none) -> LED_SMD:LED_0603_1608Metric
- IC1: footprint QFN40P700X700X90-57N-D -> SamacSys_Parts:QFN40P700X700X90-57N-D
- IC2: footprint QFN50P300X400X80-21N -> Package_DFN_QFN:Texas_RVC0020A_WQFN-20-1EP_3x4mm_P0.5mm_EP1.6x2.6mm
- IC3: footprint SOT65P210X110-6N -> SamacSys_Parts:SOT65P210X110-6N
- IC4, IC8: footprint SOT95P280X145-6N -> Package_TO_SOT_SMD:SOT-23-6
- IC5, IC6: footprint SOIC127P600X175-14N -> SamacSys_Parts:SOIC127P600X175-14N
- IC9: footprint SOP65P640X120-28N -> SamacSys_Parts:SOP65P640X120-28N
- J10, J11, J12, J13, J14, J15, J16, J5, J6, J7, J8, J9: footprint (none) -> Connector_Molex:Molex_Micro-Fit_3.0_43045-0400_2x02_P3.00mm_Horizontal
- J18: footprint RF_Module:nRF24L01_Breakout -> Connector_Molex:Molex_Micro-Fit_3.0_43045-0600_2x03_P3.00mm_Horizontal
- J2: footprint Connector_Audio:Jack_XLR_Neutrik_NC3FAAH_Horizontal -> Connector_Molex:Molex_Micro-Fit_3.0_43650-0200_1x02_P3.00mm_Horizontal
- J3: footprint Package_TO_SOT_SMD:Texas_DRT-3 -> Connector_PinHeader_2.54mm:PinHeader_1x03_P2.54mm_Vertical
- JP1: footprint PESD2CAN -> Connector_PinHeader_2.54mm:PinHeader_1x02_P2.54mm_Vertical
- L1: footprint (none) -> Inductor_SMD:L_Coilcraft_XxL4020
- L2, L3, L5, L6, L7, L8, L9: footprint (none) -> Inductor_SMD:L_0402_1005Metric
- L4: footprint (none) -> Inductor_SMD:L_0603_1608Metric
- R1, R10, R11, R12, R13, R14, R16, R17, R18, R19, R2, R20, R21, R22, R23, R24, R26, R27, R28, R29, R3, R30, R31, R32, R33, R35, R36, R37, R38, R39, R4, R40, R41, R42, R43, R44, R45, R46, R47, R48, R49, R50, R51, R52, R53, R54, R55, R56, R57, R58, R59, R6, R60, R61, R62, R63, R64, R65, R66, R67, R68, R69, R7, R70, R71, R72, R73, R74, R75, R76, R77, R78, R79, R8, R81, R84, R85, R86, R87, R9, R90, R91, R92, R93, R94: footprint (none) -> Resistor_SMD:R_0603_1608Metric
- R15: footprint Module:Arduino_UNO_R3 -> Resistor_SMD:R_0603_1608Metric
- R25: footprint (none) -> Resistor_SMD:R_0402_1005Metric
- R34: footprint Package_LCC:PLCC-84_29.3x29.3mm_P1.27mm -> Resistor_SMD:R_0603_1608Metric
- R5: footprint Package_DFN_QFN:VQFN-16-1EP_3x3mm_P0.5mm_EP1.68x1.68mm_ThermalVias -> Resistor_SMD:R_0603_1608Metric
- R80, R82, R83: footprint (none) -> Resistor_SMD:R_1206_3216Metric
- R88, R89: footprint Package_SO:TSSOP-10_3x3mm_P0.5mm -> Resistor_SMD:R_0603_1608Metric
- SW1, SW2: footprint Package_SON:WSON-8-1EP_6x5mm_P1.27mm_EP3.4x4mm -> Button_Switch_SMD:SW_Tactile_SPST_NO_Straight_CK_PTS636Sx25SMTRLFS
- U6: value MCP3208 -> MCP3208-BI/SL; footprint Package_DFN_QFN:QFN-20-1EP_5x5mm_P0.65mm_EP3.35x3.35mm -> Package_SO:SOIC-16_3.9x9.9mm_P1.27mm
