File: kicad/rtlm/rtlm.kicad_sch (KiCad schematic)
At the start: 264 parts, among them IC1 ESP32-S3FN8, IC2 TPS25940ARVCR, IC3 PE4259, IC4 TPS2553DBVR, IC5 TLV9004IDR, IC6 TLV9004IDR, IC7 TCAN1042HGVDR, IC8 TPS2553DBVR, IC9 TLC59116IPWR, J1 USB_C_Receptacle_USB2.0_16P, J10 TEMP_2, J11 TEMP_3, J12 TEMP_4, J13 ANALOG_1, J14 ANALOG_2, J15 ANALOG_3, J16 ANALOG_4, J17 DM3AT-SF-PEJM5, J18 CAN_EXPANSION, J19 BATTERY_VOLTAGE_SENSE_LINE, J2 Conn_01x02, J3 UART_DEBUG_3V3, J4 LORA_ANT, J5 PULSE_1, J6 PULSE_2, J7 PULSE_3, J8 PULSE_4, J9 TEMP_1, Q1 DMP2035U-7, SW1 SW_Push, SW2 SW_Push, U1 TPS62130A, U10 RV-3028-C7, U2 TPS2116DRL, U3 TPD2EUSB30, U4 SX1262IMLTRT, U5 SN74LVC14ADR, U6 MCP3208-BI/SL, U7 REF3025AIDBZR, U8 AMC3330, U9 ADS1115IDGS, Y1 40MHz, Y2 TG2520SMN 32.0000M-MCGNNM3

Commit message: feat: prelim RF
Parts:
- added FB1: 600R@100MHz, Inductor_SMD:L_0603_1608Metric, symbol Device:FerriteBead
- C24: MPN (none) -> GJM1555C1H100JB01D; Manufacturer (none) -> Murata
- C27, C32: MPN (none) -> GJM1555C1H390JB01D; Manufacturer (none) -> Murata
- C28: MPN (none) -> GJM1555C1H2R4BB01D; Manufacturer (none) -> Murata
- C29, C37: MPN (none) -> GJM1555C1H1R8BB01D; Manufacturer (none) -> Murata
- C30, C31: MPN (none) -> GJM1555C1H3R3BB01D; Manufacturer (none) -> Murata
- C33: MPN (none) -> GRM155R71C473KA01D; Manufacturer (none) -> Murata
- C34: MPN (none) -> GJM1555C1H470JB01D; Manufacturer (none) -> Murata
- C35: MPN (none) -> GJM1555C1H3R0BB01D; Manufacturer (none) -> Murata
- C36: MPN (none) -> GJM1555C1H5R6CB01D; Manufacturer (none) -> Murata
- L4: footprint Inductor_SMD:L_0603_1608Metric -> Inductor_SMD:L_0805_2012Metric; MPN (none) -> MLZ2012M150WT000; Manufacturer (none) -> TDK
- L5: MPN (none) -> LQW15AN15NH00D; Manufacturer (none) -> Murata
- L6: MPN (none) -> LQW15AN9N1H00D; Manufacturer (none) -> Murata
- L7: MPN (none) -> LQW15AN2N5C00D; Manufacturer (none) -> Murata
- L8: MPN (none) -> LQW15AN4N7C00D; Manufacturer (none) -> Murata
- L9: MPN (none) -> 0402HP-47NXJRW; Manufacturer (none) -> Coilcraft
Connections:
- net LORA_3V0: now also FB1.1; no longer C23.2, Y2.4 (Vcc)
- new net TCXO_3V0: C23.2, FB1.2, Y2.4 (Vcc)
Changed lines of the file:
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@@
 	(wire
 		(pts
-			(xy 294.64 137.16) (xy 317.5 137.16)
-		)
-		(stroke
-			(width 0)
-			(type default)
-		)
-	)
-	(wire
-		(pts
 			(xy 166.37 199.39) (xy 168.91 199.39)
 		)
@@
 	)
 	(label "LORA_3V0"
-		(at 307.34 137.16 270)
+		(at 317.5 137.16 0)
 		(effects
 			(font
@@
 			)
 		)
+		(property "MPN" "GJM1555C1H1R8BB01D" (at 0 0 0) (hide yes) (effects (font (size 1.27 1.27))))
+		(property "Manufacturer" "Murata" (at 0 0 0) (hide yes) (effects (font (size 1.27 1.27))))
 		(pin "2"
 		)
@@
 			)
 		)
+		(property "MPN" "GRM155R71C473KA01D" (at 0 0 0) (hide yes) (effects (font (size 1.27 1.27))))
+		(property "Manufacturer" "Murata" (at 0 0 0) (hide yes) (effects (font (size 1.27 1.27))))
 		(pin "2"
 		)
@@
 			)
 		)
+		(property "MPN" "GJM1555C1H3R3BB01D" (at 0 0 0) (hide yes) (effects (font (size 1.27 1.27))))
+		(property "Manufacturer" "Murata" (at 0 0 0) (hide yes) (effects (font (size 1.27 1.27))))
 		(pin "1"
 		)
@@
 			)
 		)
+		(property "MPN" "LQW15AN4N7C00D" (at 0 0 0) (hide yes) (effects (font (size 1.27 1.27))))
+		(property "Manufacturer" "Murata" (at 0 0 0) (hide yes) (effects (font (size 1.27 1.27))))
 		(pin "2"
 		)
@@
 			)
 		)
+		(property "MPN" "GJM1555C1H1R8BB01D" (at 0 0 0) (hide yes) (effects (font (size 1.27 1.27))))
+		(property "Manufacturer" "Murata" (at 0 0 0) (hide yes) (effects (font (size 1.27 1.27))))
 		(pin "2"
 		)
@@
 			)
 		)
+		(property "MPN" "LQW15AN15NH00D" (at 0 0 0) (hide yes) (effects (font (size 1.27 1.27))))
+		(property "Manufacturer" "Murata" (at 0 0 0) (hide yes) (effects (font (size 1.27 1.27))))
 		(pin "2"
 		)
@@
 			)
 		)
+		(property "MPN" "GJM1555C1H100JB01D" (at 0 0 0) (hide yes) (effects (font (size 1.27 1.27))))
+		(property "Manufacturer" "Murata" (at 0 0 0) (hide yes) (effects (font (size 1.27 1.27))))
 		(pin "2"
 		)
@@
 			)
 		)
+		(property "MPN" "LQW15AN9N1H00D" (at 0 0 0) (hide yes) (effects (font (size 1.27 1.27))))
+		(property "Manufacturer" "Murata" (at 0 0 0) (hide yes) (effects (font (size 1.27 1.27))))
 		(pin "2"
 		)
@@
 			)
 		)
-		(property "Footprint" "Inductor_SMD:L_0603_1608Metric"
+		(property "Footprint" "Inductor_SMD:L_0805_2012Metric"
 			(at 353.06 118.11 0)
 			(hide yes)
@@
 			)
 		)
+		(property "MPN" "MLZ2012M150WT000" (at 0 0 0) (hide yes) (effects (font (size 1.27 1.27))))
+		(property "Manufacturer" "TDK" (at 0 0 0) (hide yes) (effects (font (size 1.27 1.27))))
 		(pin "2"
 		)
@@
 			)
 		)
+		(property "MPN" "GJM1555C1H3R3BB01D" (at 0 0 0) (hide yes) (effects (font (size 1.27 1.27))))
+		(property "Manufacturer" "Murata" (at 0 0 0) (hide yes) (effects (font (size 1.27 1.27))))
 		(pin "1"
 		)
@@
 			)
 		)
+		(property "MPN" "GJM1555C1H2R4BB01D" (at 0 0 0) (hide yes) (effects (font (size 1.27 1.27))))
+		(property "Manufacturer" "Murata" (at 0 0 0) (hide yes) (effects (font (size 1.27 1.27))))
 		(pin "2"
 		)
@@
 			)
 		)
+		(property "MPN" "GJM1555C1H470JB01D" (at 0 0 0) (hide yes) (effects (font (size 1.27 1.27))))
+		(property "Manufacturer" "Murata" (at 0 0 0) (hide yes) (effects (font (size 1.27 1.27))))
 		(pin "2"
 		)
@@
 			)
 		)
+		(property "MPN" "GJM1555C1H5R6CB01D" (at 0 0 0) (hide yes) (effects (font (size 1.27 1.27))))
+		(property "Manufacturer" "Murata" (at 0 0 0) (hide yes) (effects (font (size 1.27 1.27))))
 		(pin "2"
 		)
@@
 			)
 		)
+		(property "MPN" "GJM1555C1H390JB01D" (at 0 0 0) (hide yes) (effects (font (size 1.27 1.27))))
+		(property "Manufacturer" "Murata" (at 0 0 0) (hide yes) (effects (font (size 1.27 1.27))))
 		(pin "2"
 		)
@@
 			)
 		)
+		(property "MPN" "GJM1555C1H3R0BB01D" (at 0 0 0) (hide yes) (effects (font (size 1.27 1.27))))
+		(property "Manufacturer" "Murata" (at 0 0 0) (hide yes) (effects (font (size 1.27 1.27))))
 		(pin "1"
 		)
@@
 			)
 		)
+		(property "MPN" "GJM1555C1H390JB01D" (at 0 0 0) (hide yes) (effects (font (size 1.27 1.27))))
+		(property "Manufacturer" "Murata" (at 0 0 0) (hide yes) (effects (font (size 1.27 1.27))))
 		(pin "1"
 		)
@@
 			)
 		)
+		(property "MPN" "LQW15AN2N5C00D" (at 0 0 0) (hide yes) (effects (font (size 1.27 1.27))))
+		(property "Manufacturer" "Murata" (at 0 0 0) (hide yes) (effects (font (size 1.27 1.27))))
 		(pin "1"
 		)
@@
 			)
 		)
+		(property "MPN" "0402HP-47NXJRW" (at 0 0 0) (hide yes) (effects (font (size 1.27 1.27))))
+		(property "Manufacturer" "Coilcraft" (at 0 0 0) (hide yes) (effects (font (size 1.27 1.27))))
 		(pin "2"
 		)
@@
 		)
 		(property "Value" "100nf"
-			(at 298.45 134.6199 0)
+			(at 298.45 133.985 0)
 			(show_name no)
 			(do_not_autoplace no)
@@
 	(label "5V_SYS" (at 511.81 241.3 0) (effects (font (size 1.27 1.27)) (justify right bottom)))
 	(label "GND" (at 519.43 241.3 0) (effects (font (size 1.27 1.27)) (justify left bottom)))
+	(symbol
+		(lib_id "Device:FerriteBead")
+		(at 279.4 161.29 90)
+		(unit 1)
+		(body_style 1)
+		(exclude_from_sim no)
+		(in_bom yes)
+		(on_board yes)
+		(in_pos_files yes)
+		(dnp no)
+		(fields_autoplaced yes)
+		(property "Reference" "FB1"
+			(at 279.4 156.21 90)
+			(show_name no)
+			(do_not_autoplace no)
+			(effects
+				(font
+					(size 1.27 1.27)
+				)
+				(justify left)
+			)
+		)
+		(property "Value" "600R@100MHz"
+			(at 279.4 166.37 90)
+			(show_name no)
+			(do_not_autoplace no)
+			(effects
+				(font
+					(size 1.27 1.27)
+				)
+				(justify left)
+			)
+		)
+		(property "Footprint" "Inductor_SMD:L_0603_1608Metric"
+			(at 279.4 161.29 0)
+			(hide yes)
+			(show_name no)
+			(do_not_autoplace no)
+			(effects
+				(font
+					(size 1.27 1.27)
+				)
+			)
+		)
+		(property "Datasheet" "https://www.murata.com/en-global/products/productdata/8796738650142/ENFA0003.pdf"
+			(at 279.4 161.29 0)
+			(hide yes)
+			(show_name no)
+			(do_not_autoplace no)
+			(effects
+				(font
+					(size 1.27 1.27)
+				)
+			)
+		)
+		(property "Description" "TCXO supply ferrite; Murata BLM18AG601SN1D; 600 ohm at 100MHz; 500mA; DCR <=0.38 ohm"
+			(at 279.4 161.29 0)
+			(hide yes)
+			(show_name no)
+			(do_not_autoplace no)
+			(effects
+				(font
+					(size 1.27 1.27)
+				)
+			)
+		)
+		(property "MPN" "BLM18AG601SN1D" (at 279.4 161.29 0) (effects (font (size 1.27 1.27)) (hide yes)))
+		(property "Manufacturer" "Murata" (at 0 0 0) (hide yes) (effects (font (size 1.27 1.27))))
+		(pin "2"
+		)
+		(pin "1"
+		)
+		(instances
+			(project "rtlm"
+				(path "/18642f86-b1da-4982-a59b-b3bbb269065a"
+					(reference "FB1")
+					(unit 1)
+				)
+			)
+		)
+	)
+	(label "TCXO_3V0" (at 294.64 137.16 0) (effects (font (size 1.27 1.27)) (justify left bottom)))
+	(label "LORA_3V0" (at 275.59 161.29 0) (effects (font (size 1.27 1.27)) (justify right bottom)))
+	(label "TCXO_3V0" (at 283.21 161.29 0) (effects (font (size 1.27 1.27)) (justify left bottom)))
 )

Commit message: Refine manufacturing layout and specify prototype BOM
Parts:
- BT1: MPN (none) -> 1060; Manufacturer (none) -> Keystone; Selection Notes (none) -> CR2032 holder; primary cell supplied separately; RTC chargi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
- C1: value 10µf -> 22uF; MPN (none) -> GRM21BR61E226ME44L; Manufacturer (none) -> Murata
- C10, C11, C12, C14, C15, C2, C39, C46, C49, C50, C51, C52, C53, C58, C59, C61, C62, C63, C68, C73, C76, C78, C79, C8: MPN (none) -> CC0603KRX7R9BB104; Manufacturer (none) -> Yageo; Selection Notes (none) -> Specified MLCC value/package; manufacturer datasheet and DC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
- C13, C18, C38, C42, C48, C5, C6, C66, C69, C77, C9: MPN (none) -> CC0603KRX7R8BB105; Manufacturer (none) -> Yageo; Selection Notes (none) -> Specified MLCC value/package; manufacturer datasheet and DC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
- C16, C44, C60, C65: MPN (none) -> GRM21BZ71E106KE15L; Manufacturer (none) -> Murata; Selection Notes (none) -> 10uF 25V X7R 10%; normal bypass/storage, verify transient r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
- C17: MPN (none) -> GRM188R71C105KA12D; Manufacturer (none) -> Murata
- C19, C20: MPN (none) -> GRM1885C1H160JA01D; Manufacturer (none) -> Murata
- C21, C23, C26: MPN (none) -> CC0402KRX7R9BB104; Manufacturer (none) -> Yageo; Selection Notes (none) -> Specified MLCC value/package; manufacturer datasheet and DC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
- C22: MPN (none) -> CC0402KRX5R6BB474; Manufacturer (none) -> Yageo; Selection Notes (none) -> Specified MLCC value/package; manufacturer datasheet and DC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
- C25: MPN (none) -> CC0402JRNPO9BN102; Manufacturer (none) -> Yageo; Selection Notes (none) -> Specified MLCC value/package; manufacturer datasheet and DC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
- C3: MPN (none) -> GRM31CR71A226KE15L; Manufacturer (none) -> Murata
- C4: MPN (none) -> CC0603KRX7R9BB332; Manufacturer (none) -> Yageo; Selection Notes (none) -> Specified MLCC value/package; manufacturer datasheet and DC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
- C40, C41, C43, C45, C70: MPN (none) -> CC0603JRNPO9BN102; Manufacturer (none) -> Yageo; Selection Notes (none) -> Specified MLCC value/package; manufacturer datasheet and DC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
- C47: MPN (none) -> CC0603KRX7R7BB474; Manufacturer (none) -> Yageo; Selection Notes (none) -> Specified MLCC value/package; manufacturer datasheet and DC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
- C54, C55, C56, C57, C7, C75: MPN (none) -> CC0603KRX7R9BB103; Manufacturer (none) -> Yageo; Selection Notes (none) -> Specified MLCC value/package; manufacturer datasheet and DC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
- C64: MPN (none) -> CC1206KKX7R9BB105; Manufacturer (none) -> Yageo; Selection Notes (none) -> Specified MLCC value/package; manufacturer datasheet and DC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
- C67, C72: MPN (none) -> CC1206JRNPO9BN102; Manufacturer (none) -> Yageo; Selection Notes (none) -> Specified MLCC value/package; manufacturer datasheet and DC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
- C71: MPN (none) -> CC1206KRX7R9BB104; Manufacturer (none) -> Yageo; Selection Notes (none) -> Specified MLCC value/package; manufacturer datasheet and DC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
- C74: MPN (none) -> CC0603KRX7R0BB103; Manufacturer (none) -> Yageo; Selection Notes (none) -> 10nF 100V X7R 10% divider filter; voltage headroom for open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
- C80, C81: value 10uF -> 22uF; MPN (none) -> GRM21BR61E226ME44L; Manufacturer (none) -> Murata
- D1: MPN (none) -> BZT52C5V6-7-F; Manufacturer (none) -> Diodes Incorporated; Selection Notes (none) -> 5.6V SOD123 gate protection zener.
- D18, D20, D21, D22, D23, D24, D25, D26, D27, D28, D29, D30, D31, D32, D33, D34: MPN (none) -> APT1608SGC; Manufacturer (none) -> Kingbright
- D2, D4, D6, D8: MPN (none) -> PESD5V0S1UL,315; Manufacturer (none) -> Nexperia; Selection Notes (none) -> 5V ESD diode SOD882.
- D3, D5, D7, D9: MPN (none) -> BAT54S,215; Manufacturer (none) -> Nexperia; Selection Notes (none) -> Dual series Schottky clamp, SOT23.
- IC1: footprint SamacSys_Parts:QFN40P700X700X90-57N-D -> RTLM_Local:ESP32_S3_QFN56_EP_Windowed
- J1: footprint Connector_USB:USB_C_Receptacle_GCT_USB4105-xx-A_16P_TopMnt_Horizontal -> RTLM_Local:USB_C_GCT_USB4105_JLC_NPTH_Clearance; MPN (none) -> USB4105-GF-A; Manufacturer (none) -> GCT; Selection Notes (none) -> USB4105 top-mount USB2 Type-C; verify selected staking leng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
- J10, J11, J12, J13, J14, J15, J16, J5, J6, J7, J8, J9: MPN (none) -> 430450400; Manufacturer (none) -> Molex; Selection Notes (none) -> Micro-Fit 3.0 2x2 right-angle; connector pinout table defin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
- J17: MPN (none) -> DM3AT-SF-PEJM5(40); Manufacturer (none) -> Hirose; Selection Notes (none) -> Push-push microSD socket; qualify a card within 400mA peak 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
- J18: MPN (none) -> 430450600; Manufacturer (none) -> Molex; Selection Notes (none) -> Micro-Fit 3.0 2x3 right-angle CAN expansion.
- J19: MPN (none) -> 436500300; Manufacturer (none) -> Molex; Selection Notes (none) -> Micro-Fit 3.0 1x3 right-angle pack sense; center contact NC.
- J2: MPN (none) -> 436500200; Manufacturer (none) -> Molex; Selection Notes (none) -> Micro-Fit 3.0 1x2 right-angle 5V input.
- J3: MPN (none) -> TSW-103-07-G-S; Manufacturer (none) -> Samtec; Selection Notes (none) -> 2.54mm 1x3 debug header; check mating height against enclos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
- J4: MPN (none) -> U.FL-R-SMT-1(10); Manufacturer (none) -> Hirose; Selection Notes (none) -> U.FL 50Ohm board receptacle; cable/antenna specified separa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
- JP1: MPN (none) -> TSW-102-07-G-S; Manufacturer (none) -> Samtec; Selection Notes (none) -> 2.54mm 1x2 header; separate jumper shunt; enable 120Ohm onl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
- L1: MPN (none) -> XAL4020-222MEC; Manufacturer (none) -> Coilcraft
- L2: MPN (none) -> 0402HP-2N0XJRW; Manufacturer (none) -> Coilcraft
- L3: MPN (none) -> 0402HP-24NXJRW; Manufacturer (none) -> Coilcraft
- Q1: MPN (none) -> DMP2035U-7; Manufacturer (none) -> Diodes Incorporated; Selection Notes (none) -> P-channel SOT23 reverse-polarity MOSFET; verify hot loss in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
- R1, R2: MPN (none) -> RC0603FR-075K1L; Manufacturer (none) -> Yageo; Selection Notes (none) -> 1% standard thick film; 0Ohm jumper where value is zero.
- R10, R35, R8: MPN (none) -> RC0603FR-07100KL; Manufacturer (none) -> Yageo; Selection Notes (none) -> 1% standard thick film; 0Ohm jumper where value is zero.
- R11: MPN (none) -> RC0603FR-0742K2L; Manufacturer (none) -> Yageo; Selection Notes (none) -> 1% standard thick film; 0Ohm jumper where value is zero.
- R12: MPN (none) -> TNPW060344K2BEEA; Manufacturer (none) -> Vishay; Selection Notes (none) -> 0.1% 25ppm/K precision resistor; preserve specified divider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
- R13, R38, R41, R43, R45, R52, R54, R57, R60, R67: MPN (none) -> TNPW060310K0BEEA; Manufacturer (none) -> Vishay; Selection Notes (none) -> 0.1% 25ppm/K precision resistor; preserve specified divider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
- R14: MPN (none) -> RC0603FR-0734K8L; Manufacturer (none) -> Yageo; Selection Notes (none) -> 1% standard thick film; 0Ohm jumper where value is zero.
- R15, R16, R17, R18, R19, R21, R36, R37, R68, R69, R70, R71, R72, R74, R79, R9, R91, R93: MPN (none) -> RC0603FR-0710KL; Manufacturer (none) -> Yageo; Selection Notes (none) -> 1% standard thick film; 0Ohm jumper where value is zero.
- R20: MPN (none) -> RC0603FR-07499RL; Manufacturer (none) -> Yageo; Selection Notes (none) -> 1% standard thick film; 0Ohm jumper where value is zero.
- R22, R23: MPN (none) -> RC0603FR-07220RL; Manufacturer (none) -> Yageo; Selection Notes (none) -> 1% standard thick film; 0Ohm jumper where value is zero.
- R24, R85: MPN (none) -> RC0603FR-072K2L; Manufacturer (none) -> Yageo; Selection Notes (none) -> 1% standard thick film; 0Ohm jumper where value is zero.
- R25: MPN (none) -> RC0402JR-070RL; Manufacturer (none) -> Yageo; Selection Notes (none) -> 1% standard thick film; 0Ohm jumper where value is zero.
- R26, R29, R31, R33, R75, R76, R77, R78, R90, R94: MPN (none) -> RC0603FR-071KL; Manufacturer (none) -> Yageo; Selection Notes (none) -> 1% standard thick film; 0Ohm jumper where value is zero.
- R27, R28, R30, R32, R39, R42, R44, R46, R51, R55, R58, R61, R88, R89: MPN (none) -> RC0603FR-074K7L; Manufacturer (none) -> Yageo; Selection Notes (none) -> 1% standard thick film; 0Ohm jumper where value is zero.
- R3, R4: MPN (none) -> RC0603FR-0722RL; Manufacturer (none) -> Yageo; Selection Notes (none) -> 1% standard thick film; 0Ohm jumper where value is zero.
- R34: MPN (none) -> RC0603FR-0752K3L; Manufacturer (none) -> Yageo; Selection Notes (none) -> 1% standard thick film; 0Ohm jumper where value is zero.
- R40, R47, R48, R49, R62, R63, R64, R65: MPN (none) -> RC0603FR-0747RL; Manufacturer (none) -> Yageo; Selection Notes (none) -> 1% standard thick film; 0Ohm jumper where value is zero.
- R5: MPN (none) -> RC0603FR-0724KL; Manufacturer (none) -> Yageo; Selection Notes (none) -> 1% standard thick film; 0Ohm jumper where value is zero.
- R50, R53, R56, R59: MPN (none) -> TNPW060312K0BEEA; Manufacturer (none) -> Vishay; Selection Notes (none) -> 0.1% 25ppm/K precision resistor; preserve specified divider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
- R6: MPN (none) -> RC0603FR-0775KL; Manufacturer (none) -> Yageo; Selection Notes (none) -> 1% standard thick film; 0Ohm jumper where value is zero.
- R66: MPN (none) -> TNPW060320K0BEEA; Manufacturer (none) -> Vishay; Selection Notes (none) -> 0.1% 25ppm/K precision resistor; preserve specified divider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
- R7: MPN (none) -> RC0603FR-0730KL; Manufacturer (none) -> Yageo; Selection Notes (none) -> 1% standard thick film; 0Ohm jumper where value is zero.
- R73: MPN (none) -> RC0603FR-0733RL; Manufacturer (none) -> Yageo; Selection Notes (none) -> 1% standard thick film; 0Ohm jumper where value is zero.
- R80: MPN (none) -> CRCW1206120RFKEAHP; Manufacturer (none) -> Vishay; Selection Notes (none) -> 120Ohm 1% 1206 high-power termination; 0.75W rating require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
- R81: MPN (none) -> RC0603FR-0788K7L; Manufacturer (none) -> Yageo; Selection Notes (none) -> 1% standard thick film; 0Ohm jumper where value is zero.
- R82, R83: MPN (none) -> TNPW1206499KBEEA; Manufacturer (none) -> Vishay
- R84: MPN (none) -> TNPW06038K20BEEA; Manufacturer (none) -> Vishay
- R86, R87: MPN (none) -> RC0603FR-07470RL; Manufacturer (none) -> Yageo; Selection Notes (none) -> 1% standard thick film; 0Ohm jumper where value is zero.
- R92: MPN (none) -> RC0603FR-071K8L; Manufacturer (none) -> Yageo; Selection Notes (none) -> 1% standard thick film; 0Ohm jumper where value is zero.
- SW1, SW2: MPN (none) -> PTS636SM25SMTRLFS; Manufacturer (none) -> C&K; Selection Notes (none) -> PTS636 2.5mm actuator; enclosure actuator alignment remains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
- U1: MPN (none) -> TPS62130ARGTR; Manufacturer (none) -> Texas Instruments; Selection Notes (none) -> Adjustable 3A buck; system budget is 1.30A, not 3A.
- U10: MPN (none) -> RV-3028-C7 32.768kHz 1ppm TA QC; Manufacturer (none) -> Micro Crystal; Selection Notes (none) -> Factory-calibrated RTC; confirm procurement packing code; n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
- U2: MPN (none) -> TPS2116DRLR; Manufacturer (none) -> Texas Instruments; Selection Notes (none) -> 2.5A power mux, DRL8.
- U3: MPN (none) -> TPD2EUSB30DRTR; Manufacturer (none) -> Texas Instruments; Selection Notes (none) -> 2-channel USB ESD protection, DRT3.
- U4: MPN (none) -> SX1262IMLTRT; Manufacturer (none) -> Semtech; Selection Notes (none) -> SX1262 QFN24; reference design 902-928MHz, conducted qualif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
- U5: MPN (none) -> SN74LVC14ADR; Manufacturer (none) -> Texas Instruments; Selection Notes (none) -> LVC hex Schmitt inverter, SOIC14; 1.65-3.6V supply, 5.5V-to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
- U6: MPN (none) -> MCP3208-BI/SL; Manufacturer (none) -> Microchip; Selection Notes (none) -> 12-bit 8-channel ADC, SOIC16; start <=1MHz SPI.
- U7: MPN (none) -> REF3025AIDBZR; Manufacturer (none) -> Texas Instruments; Selection Notes (none) -> 2.5V reference, SOT23.
- U8: footprint Package_SO:SOIC-16W_7.5x10.3mm_P1.27mm -> RTLM_Local:AMC3330_DWE0016A_HV_8p1mm; MPN (none) -> AMC3330DWER; Manufacturer (none) -> Texas Instruments; Selection Notes (none) -> AMC3330 isolated +/-1V input amplifier, DWE16; TI HV land p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
- U9: MPN (none) -> ADS1115IDGSR; Manufacturer (none) -> Texas Instruments; Selection Notes (none) -> 16-bit differential ADC, VSSOP10; +/-2.048V or wider PGA fo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
- Y1: MPN (none) -> Q22FA1280010118; Manufacturer (none) -> Epson
- Y2: MPN (none) -> TG2520SMN 32.0000M-MCGNNM3; Manufacturer (none) -> Epson; Selection Notes (none) -> 32MHz 3.0V TCXO; operating GPIO/TCXO setup required.
