File: kicad/rtlm/rtlm.kicad_sch (KiCad schematic)
At the start: 292 parts, among them IC1 ESP32-S3FN8, IC2 TPS25940ARVCR, IC3 PE4259, IC4 TPS2553DBVR, IC5 TLV9004IDR, IC6 TLV9004IDR, IC7 TCAN1042HGVDR, IC8 TPS2553DBVR, IC9 TLC59116IPWR, J1 TYPE-C-31-M-12, J10 TEMP_2, J11 TEMP_3, J12 TEMP_4, J13 ANALOG_1, J14 ANALOG_2, J15 ANALOG_3, J16 ANALOG_4, J17 DM3AT-SF-PEJM5, J18 CAN_EXPANSION, J19 BATTERY_VOLTAGE_SENSE_LINE, J2 Conn_01x02, J3 UART_DEBUG_3V3, J4 LORA_ANT, J5 PULSE_1, J6 PULSE_2, J7 PULSE_3, J8 PULSE_4, J9 TEMP_1, Q1 DMP2035U-7, Q2 MMBT3904-7-F, Q3 MMBT3904-7-F, SW1 SW_Push, SW2 SW_Push, U1 TPS62130A, U10 RV-3028-C7, U11 TPS22917DBVR, U12 TPS3808G01DBVR, U13 SN74LVC2G17DBVR, U14 SN74LVC2G86DCTR, U2 TPS2116DRL, U3 TPD2EUSB30, U4 SX1262IMLTRT, U5 SN74LVC14ADR, U6 MCP3208-BI/SL, U7 REF3025AIDBZR, U8 AMC3330, U9 ADS1115IDGS, Y1 40MHz, Y2 TG2520SMN 32.0000M-MCGNNM3

Commit message: Qualify stocked parts for five-board prototype assembly
Parts:
- C1, C80, C81: LCSC Part Number (none) -> C86816
- C10, C11, C12, C14, C15, C2, C39, C46, C49, C50, C51, C52, C53, C58, C59, C61, C62, C63, C68, C73, C76, C78, C79, C8, C82, C85, C88, C89: LCSC Part Number (none) -> C14663
- C13, C18, C38, C42, C48, C5, C6, C66, C69, C77, C83, C9: LCSC Part Number (none) -> C106858
- C16, C44, C60, C65: LCSC Part Number (none) -> C237493
- C17: LCSC Part Number (none) -> C106858; MPN GRM188R71C105KA12D -> CC0603KRX7R8BB105; Manufacturer Murata -> YAGEO; Selection Notes (none) -> 1uF +/-10%, X7R, 25V, 0603; replaces obsolete Murata 1uF 16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
- C21, C23, C26: LCSC Part Number (none) -> C131394
- C22: LCSC Part Number (none) -> C106255
- C24: LCSC Part Number (none) -> C85874
- C29, C37: LCSC Part Number (none) -> C76902
- C3: LCSC Part Number (none) -> C91604
- C30, C31: LCSC Part Number (none) -> C76906
- C33: LCSC Part Number (none) -> C77012
- C34: LCSC Part Number (none) -> C161322
- C35: LCSC Part Number (none) -> C88891
- C36: LCSC Part Number (none) -> C88895
- C4: LCSC Part Number (none) -> C106222
- C40, C41, C43, C45, C70, C84: LCSC Part Number (none) -> C106246
- C47: LCSC Part Number (none) -> C106851
- C54, C55, C56, C57, C7, C75, C90: LCSC Part Number (none) -> C100042
- C64: LCSC Part Number (none) -> C107185
- C67, C72: LCSC Part Number (none) -> C113881
- C71: LCSC Part Number (none) -> C82601
- C74: LCSC Part Number (none) -> C107059
- C87: LCSC Part Number (none) -> C107083
- D1: LCSC Part Number (none) -> C397930
- D10, D11, D12, D13, D14, D15, D16, D17: LCSC Part Number (none) -> C3001947
- D18, D20, D21, D22, D23, D24, D25, D26, D27, D28, D29, D30, D31, D32, D33, D34: LCSC Part Number (none) -> C5875754
- D19: LCSC Part Number (none) -> C284078
- D2, D4, D6, D8: LCSC Part Number (none) -> C85402
- D3, D5, D7, D9: LCSC Part Number (none) -> C47546
- F1: LCSC Part Number (none) -> C3159235
- FB1: LCSC Part Number (none) -> C19330
- IC1: LCSC Part Number (none) -> C2913196
- IC2: LCSC Part Number (none) -> C2653873
- IC3: LCSC Part Number (none) -> C470892; MPN (none) -> PE4259-63; Manufacturer (none) -> pSemi; Manufacturer_Name Peregrine Semiconductor -> pSemi; Manufacturer_Part_Number PE4259 -> PE4259-63; Selection Notes (none) -> Exact PE4259-63 SC-70-6 ordering code; use3.0V supply and e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
- IC4, IC8: LCSC Part Number (none) -> C55266
- IC5, IC6: LCSC Part Number (none) -> C2058000
- IC7: LCSC Part Number (none) -> C124014
- IC9: LCSC Part Number (none) -> C131194
- J10, J11, J12, J13, J14, J15, J16, J5, J6, J7, J8, J9: LCSC Part Number (none) -> C122413
- J17: LCSC Part Number (none) -> C597971
- J18: LCSC Part Number (none) -> C127367
- J19: LCSC Part Number (none) -> C503478
- J2: LCSC Part Number (none) -> C192562
- J3: LCSC Part Number (none) -> C3335811
- J4: LCSC Part Number (none) -> C88373
- JP1: LCSC Part Number (none) -> C7402729
- L1: LCSC Part Number (none) -> C3151182
- L4: LCSC Part Number (none) -> C383402
- L5: LCSC Part Number (none) -> C91621
- L7: LCSC Part Number (none) -> C703121
- L8: LCSC Part Number (none) -> C167480
- Q1: LCSC Part Number (none) -> C110499
- Q2, Q3: LCSC Part Number (none) -> C94514
- R1, R2: LCSC Part Number (none) -> C105580
- R10, R102, R104, R105, R35, R8, R96: LCSC Part Number (none) -> C14675
- R100: LCSC Part Number (none) -> C105588
- R101, R103, R15, R16, R17, R18, R19, R21, R36, R37, R68, R69, R70, R71, R72, R74, R79, R9, R91, R93, R98: LCSC Part Number (none) -> C98220
- R11: LCSC Part Number (none) -> C273741
- R13, R38, R41, R43, R45, R52, R54, R57, R60, R67: LCSC Part Number (none) -> C844890
- R14: LCSC Part Number (none) -> C137741
- R20: LCSC Part Number (none) -> C137714
- R22, R23: LCSC Part Number (none) -> C107696
- R24, R85: LCSC Part Number (none) -> C114662
- R25: LCSC Part Number (none) -> C60485
- R26, R29, R31, R33, R75, R76, R77, R78, R90, R94: LCSC Part Number (none) -> C22548
- R27, R28, R30, R32, R39, R42, R44, R46, R51, R55, R58, R61, R88, R89: LCSC Part Number (none) -> C99782
- R3, R4: LCSC Part Number (none) -> C107701
- R34: LCSC Part Number (none) -> C23198; MPN RC0603FR-0752K3L -> 0603WAF5232T5E; Manufacturer Yageo -> Royal Ohm; Selection Notes 1% standard thick film; 0Ohm jumper where value is zero. -> 52.3k +/-1%,0603,0.1W,100ppm/K,75V; same value and ratings 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
- R40, R47, R48, R49, R62, R63, R64, R65: LCSC Part Number (none) -> C114623
- R5: LCSC Part Number (none) -> C137760
- R6: LCSC Part Number (none) -> C114636
- R7: LCSC Part Number (none) -> C100001
- R73: LCSC Part Number (none) -> C108661
- R80: LCSC Part Number (none) -> C5578739
- R81: LCSC Part Number (none) -> C163418
- R82, R83: LCSC Part Number (none) -> C2073405
- R84: MPN TNPW060316K4BEEA -> RN73R1JTTD1642B25; Manufacturer Vishay -> KOA Speer; Selection Notes (none) -> 16.4k 0.1% 25ppm/K, 0603, 0.1W/75V. Same divider value; nor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
- R86, R87: LCSC Part Number (none) -> C114669
- R92: LCSC Part Number (none) -> C185354
- R95: MPN TNPW060316K4BEEA -> RN73R1JTTD1642B25; Manufacturer Vishay -> KOA Speer; Selection Notes Independent parallel lower divider leg, not series redundan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 -> 16.4k 0.1% 25ppm/K, 0603, 0.1W/75V. Same divider value; nor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
- R97: LCSC Part Number (none) -> C105578
- R99: LCSC Part Number (none) -> C105579
- SW1, SW2: LCSC Part Number (none) -> C2799946
- U1: LCSC Part Number (none) -> C337502
- U10: LCSC Part Number (none) -> C3019759
- U11: LCSC Part Number (none) -> C2681320
- U12: LCSC Part Number (none) -> C19653
- U14: LCSC Part Number (none) -> C130023
- U2: LCSC Part Number (none) -> C3235557
- U3: LCSC Part Number (none) -> C97502
- U4: LCSC Part Number (none) -> C191341
- U5: LCSC Part Number (none) -> C133541
- U6: LCSC Part Number (none) -> C2979740
- U7: value REF3025AIDBZR -> REF3025AIDBZT; LCSC Part Number (none) -> C96625; MPN REF3025AIDBZR -> REF3025AIDBZT; Selection Notes 2.5V reference, SOT23. -> Same REF3025A DBZ SOT-23 device; small-reel T instead of R.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
- U8: LCSC Part Number (none) -> C2999368
- U9: value ADS1115IDGS -> ADS1115IDGST; LCSC Part Number (none) -> C468683; MPN ADS1115IDGSR -> ADS1115IDGST; Selection Notes 16-bit differential ADC, VSSOP10; +/-2.048V or wider PGA fo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 -> Same ADS1115 DGS VSSOP-10 device; small-reel T instead of R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
- Y1: MPN Q22FA1280010118 -> FA-128 40.0000MF20X-K0; Selection Notes (none) -> Orderable Epson FA-128 40MHz, CL10pF, +/-10ppm initial, +/-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
- Y2: value TG2520SMN 32.0000M-MCGNNM3 -> ECS-TXO-25CSMV-320-AN-TR; footprint Oscillator:Oscillator_SMD_SeikoEpson_TG2520SMN-xxx-xxxxxx-4Pin_2.5x2.0mm -> Oscillator:Oscillator_SMD_ECS_2520MV-xxx-xx-4Pin_2.5x2.0mm; symbol Oscillator:TG2520SMN-xx.xxxxxxMhz-xxxxNM -> RTLM_Local:ECS-TXO-25CSMV-320-AN-TR; MPN TG2520SMN 32.0000M-MCGNNM3 -> ECS-TXO-25CSMV-320-AN-TR; Manufacturer Epson -> ECS Inc.; Selection Notes 32MHz 3.0V TCXO; operating GPIO/TCXO setup required. -> 32MHz clipped sine, +/-0.5ppm stability, -40..85C,1.7..3.46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
Connections:
- net GND: now also Y2.1 (GND)
